Commit message: cameras working and environment resized

File: resources/models/environment_assets/walls/back_wall.urdf (robot description, URDF)
Before this commit: robot back_wall, 1 links, 0 joints
Links:
- link base_link: geometry collision box size=0.2 5.0 5.0; visual box size=0.2 5.0 5.0

File: resources/models/environment_assets/walls/front_wall.urdf (robot description, URDF)
Before this commit: robot front_wall, 1 links, 0 joints
Links:
- link base_link: geometry collision box size=0.2 5.0 5.0; visual box size=0.2 5.0 5.0

File: resources/models/environment_assets/walls/left_wall.urdf (robot description, URDF)
Before this commit: robot left_wall, 1 links, 0 joints
Links:
- link base_link: geometry collision box size=10 0.2 5; visual box size=10 0.2 5

File: resources/models/environment_assets/walls/right_wall.urdf (robot description, URDF)
Before this commit: robot right_wall, 1 links, 0 joints
Links:
- link base_link: geometry collision box size=10 0.2 5; visual box size=10 0.2 5
