Commit message: Aggiunti limiti di velocità e reward modificata. Si schianta

File: resources/models/obstacles/objects/small_sphere.urdf (robot description, URDF)
Before this commit: robot sphere, 1 links, 0 joints
Links:
- link base_link: geometry collision sphere radius=0.1; visual sphere radius=0.1
